File: hardware/lcd_board_hdmi.kicad_sch (KiCad schematic)
At the start: 32 parts, among them J1 HDMI-A receptacle, U1 LT8619C, Y1 25MHz 12pF

Commit message: Use 0603 passives and remove the alternative touch connector J6
- All 0402 resistors/capacitors are now 0603 (LCSC numbers updated to the
  matching 0603 basic parts); bulk/high-voltage caps stay 0805/1206
- J6 (JST-SH touch header) removed
- LT8619C decoupling pre-routes, crystal and REXT placement adapted to the
  larger footprints; RGB bus escape area under the chip kept free
- Re-routed (Freerouting 2.0.1), DRC: 0 errors, 0 unconnected
- Schematic, BOM/CPL, gerbers, images and README regenerated

Co-Authored-By: Claude Opus 5.5 <noreply@anthropic.com>
Claude-Session: https://claude.ai/code/session_01X8BrieHZtCS6HfoR48ML9y
Parts:
- C10, C9: footprint Capacitor_SMD:C_0402_1005Metric -> Capacitor_SMD:C_0603_1608Metric
- C11, C12, C13, C14, C15, C16, C17, C18, C19, C20, C21, C22, C23, C24: footprint Capacitor_SMD:C_0402_1005Metric -> Capacitor_SMD:C_0603_1608Metric; LCSC C1525 -> C14663
- R10, R11, R5, R6, R8, R9: footprint Resistor_SMD:R_0402_1005Metric -> Resistor_SMD:R_0603_1608Metric
- R12: footprint Resistor_SMD:R_0402_1005Metric -> Resistor_SMD:R_0603_1608Metric; LCSC C25744 -> C25804
- R13, R14: footprint Resistor_SMD:R_0402_1005Metric -> Resistor_SMD:R_0603_1608Metric; LCSC C25900 -> C23162
- R3: footprint Resistor_SMD:R_0402_1005Metric -> Resistor_SMD:R_0603_1608Metric; LCSC C11702 -> C21190
- R4: footprint Resistor_SMD:R_0402_1005Metric -> Resistor_SMD:R_0603_1608Metric; LCSC C25741 -> C25803
Changed lines of the file:
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@@
         (font
           (size 1.27 1.27))))
-    (property "Footprint" "Resistor_SMD:R_0402_1005Metric"
+    (property "Footprint" "Resistor_SMD:R_0603_1608Metric"
       (at 187.96 39.37 0)
       (effects
@@
         (font
           (size 1.27 1.27)) hide))
-    (property "LCSC" "C11702"
+    (property "LCSC" "C21190"
       (at 187.96 39.37 0)
       (effects
@@
         (font
           (size 1.27 1.27))))
-    (property "Footprint" "Resistor_SMD:R_0402_1005Metric"
+    (property "Footprint" "Resistor_SMD:R_0603_1608Metric"
       (at 220.98 39.37 0)
       (effects
@@
         (font
           (size 1.27 1.27)) hide))
-    (property "LCSC" "C25741"
+    (property "LCSC" "C25803"
       (at 220.98 39.37 0)
       (effects
@@
         (font
           (size 1.27 1.27))))
-    (property "Footprint" "Resistor_SMD:R_0402_1005Metric"
+    (property "Footprint" "Resistor_SMD:R_0603_1608Metric"
       (at 255.27 39.37 0)
       (effects
@@
         (font
           (size 1.27 1.27))))
-    (property "Footprint" "Resistor_SMD:R_0402_1005Metric"
+    (property "Footprint" "Resistor_SMD:R_0603_1608Metric"
       (at 289.56 39.37 0)
       (effects
@@
         (font
           (size 1.27 1.27))))
-    (property "Footprint" "Resistor_SMD:R_0402_1005Metric"
+    (property "Footprint" "Resistor_SMD:R_0603_1608Metric"
       (at 325.12 39.37 0)
       (effects
@@
         (font
           (size 1.27 1.27))))
-    (property "Footprint" "Resistor_SMD:R_0402_1005Metric"
+    (property "Footprint" "Resistor_SMD:R_0603_1608Metric"
       (at 30.48 168.91 0)
       (effects
@@
         (font
           (size 1.27 1.27))))
-    (property "Footprint" "Resistor_SMD:R_0402_1005Metric"
+    (property "Footprint" "Resistor_SMD:R_0603_1608Metric"
       (at 66.04 168.91 0)
       (effects
@@
         (font
           (size 1.27 1.27))))
-    (property "Footprint" "Resistor_SMD:R_0402_1005Metric"
+    (property "Footprint" "Resistor_SMD:R_0603_1608Metric"
       (at 99.06 168.91 0)
       (effects
@@
         (font
           (size 1.27 1.27))))
-    (property "Footprint" "Resistor_SMD:R_0402_1005Metric"
+    (property "Footprint" "Resistor_SMD:R_0603_1608Metric"
       (at 132.08 168.91 0)
       (effects
@@
         (font
           (size 1.27 1.27)) hide))
-    (property "LCSC" "C25744"
+    (property "LCSC" "C25804"
       (at 132.08 168.91 0)
       (effects
@@
         (font
           (size 1.27 1.27))))
-    (property "Footprint" "Resistor_SMD:R_0402_1005Metric"
+    (property "Footprint" "Resistor_SMD:R_0603_1608Metric"
       (at 162.56 168.91 0)
       (effects
@@
         (font
           (size 1.27 1.27)) hide))
-    (property "LCSC" "C25900"
+    (property "LCSC" "C23162"
       (at 162.56 168.91 0)
       (effects
@@
         (font
           (size 1.27 1.27))))
-    (property "Footprint" "Resistor_SMD:R_0402_1005Metric"
+    (property "Footprint" "Resistor_SMD:R_0603_1608Metric"
       (at 193.04 168.91 0)
       (effects
@@
         (font
           (size 1.27 1.27)) hide))
-    (property "LCSC" "C25900"
+    (property "LCSC" "C23162"
       (at 193.04 168.91 0)
       (effects
@@
         (font
           (size 1.27 1.27))))
-    (property "Footprint" "Capacitor_SMD:C_0402_1005Metric"
+    (property "Footprint" "Capacitor_SMD:C_0603_1608Metric"
       (at 222.25 168.91 0)
       (effects
@@
         (font
           (size 1.27 1.27))))
-    (property "Footprint" "Capacitor_SMD:C_0402_1005Metric"
+    (property "Footprint" "Capacitor_SMD:C_0603_1608Metric"
       (at 250.19 168.91 0)
       (effects
@@
         (font
           (size 1.27 1.27))))
-    (property "Footprint" "Capacitor_SMD:C_0402_1005Metric"
+    (property "Footprint" "Capacitor_SMD:C_0603_1608Metric"
       (at 278.13 168.91 0)
       (effects
@@
         (font
           (size 1.27 1.27)) hide))
-    (property "LCSC" "C1525"
+    (property "LCSC" "C14663"
       (at 278.13 168.91 0)
       (effects
@@
         (font
           (size 1.27 1.27))))
-    (property "Footprint" "Capacitor_SMD:C_0402_1005Metric"
+    (property "Footprint" "Capacitor_SMD:C_0603_1608Metric"
       (at 306.07 168.91 0)
       (effects
@@
         (font
           (size 1.27 1.27)) hide))
-    (property "LCSC" "C1525"
+    (property "LCSC" "C14663"
       (at 306.07 168.91 0)
       (effects
@@
         (font
           (size 1.27 1.27))))
-    (property "Footprint" "Capacitor_SMD:C_0402_1005Metric"
+    (property "Footprint" "Capacitor_SMD:C_0603_1608Metric"
       (at 334.01 168.91 0)
       (effects
@@
         (font
           (size 1.27 1.27)) hide))
-    (property "LCSC" "C1525"
+    (property "LCSC" "C14663"
       (at 334.01 168.91 0)
       (effects
@@
         (font
           (size 1.27 1.27))))
-    (property "Footprint" "Capacitor_SMD:C_0402_1005Metric"
+    (property "Footprint" "Capacitor_SMD:C_0603_1608Metric"
       (at 361.95 168.91 0)
       (effects
@@
         (font
           (size 1.27 1.27)) hide))
-    (property "LCSC" "C1525"
+    (property "LCSC" "C14663"
       (at 361.95 168.91 0)
       (effects
@@
         (font
           (size 1.27 1.27))))
-    (property "Footprint" "Capacitor_SMD:C_0402_1005Metric"
+    (property "Footprint" "Capacitor_SMD:C_0603_1608Metric"
       (at 25.4 187.96 0)
       (effects
@@
         (font
           (size 1.27 1.27)) hide))
-    (property "LCSC" "C1525"
+    (property "LCSC" "C14663"
       (at 25.4 187.96 0)
       (effects
@@
         (font
           (size 1.27 1.27))))
-    (property "Footprint" "Capacitor_SMD:C_0402_1005Metric"
+    (property "Footprint" "Capacitor_SMD:C_0603_1608Metric"
       (at 53.34 187.96 0)
       (effects
@@
         (font
           (size 1.27 1.27)) hide))
-    (property "LCSC" "C1525"
+    (property "LCSC" "C14663"
       (at 53.34 187.96 0)
       (effects
@@
         (font
           (size 1.27 1.27))))
-    (property "Footprint" "Capacitor_SMD:C_0402_1005Metric"
+    (property "Footprint" "Capacitor_SMD:C_0603_1608Metric"
       (at 78.74 187.96 0)
       (effects
@@
         (font
           (size 1.27 1.27)) hide))
-    (property "LCSC" "C1525"
+    (property "LCSC" "C14663"
       (at 78.74 187.96 0)
       (effects
@@
         (font
           (size 1.27 1.27))))
-    (property "Footprint" "Capacitor_SMD:C_0402_1005Metric"
+    (property "Footprint" "Capacitor_SMD:C_0603_1608Metric"
       (at 105.41 187.96 0)
       (effects
@@
         (font
           (size 1.27 1.27)) hide))
-    (property "LCSC" "C1525"
+    (property "LCSC" "C14663"
       (at 105.41 187.96 0)
       (effects
@@
         (font
           (size 1.27 1.27))))
-    (property "Footprint" "Capacitor_SMD:C_0402_1005Metric"
+    (property "Footprint" "Capacitor_SMD:C_0603_1608Metric"
       (at 130.81 187.96 0)
       (effects
@@
         (font
           (size 1.27 1.27)) hide))
-    (property "LCSC" "C1525"
+    (property "LCSC" "C14663"
       (at 130.81 187.96 0)
       (effects
@@
         (font
           (size 1.27 1.27))))
-    (property "Footprint" "Capacitor_SMD:C_0402_1005Metric"
+    (property "Footprint" "Capacitor_SMD:C_0603_1608Metric"
       (at 157.48 187.96 0)
       (effects
@@
         (font
           (size 1.27 1.27)) hide))
-    (property "LCSC" "C1525"
+    (property "LCSC" "C14663"
       (at 157.48 187.96 0)
       (effects
@@
         (font
           (size 1.27 1.27))))
-    (property "Footprint" "Capacitor_SMD:C_0402_1005Metric"
+    (property "Footprint" "Capacitor_SMD:C_0603_1608Metric"
       (at 184.15 187.96 0)
       (effects
@@
         (font
           (size 1.27 1.27)) hide))
-    (property "LCSC" "C1525"
+    (property "LCSC" "C14663"
       (at 184.15 187.96 0)
       (effects
@@
         (font
           (size 1.27 1.27))))
-    (property "Footprint" "Capacitor_SMD:C_0402_1005Metric"
+    (property "Footprint" "Capacitor_SMD:C_0603_1608Metric"
       (at 210.82 187.96 0)
       (effects
@@
         (font
           (size 1.27 1.27)) hide))
-    (property "LCSC" "C1525"
+    (property "LCSC" "C14663"
       (at 210.82 187.96 0)
       (effects
@@
         (font
           (size 1.27 1.27))))
-    (property "Footprint" "Capacitor_SMD:C_0402_1005Metric"
+    (property "Footprint" "Capacitor_SMD:C_0603_1608Metric"
       (at 237.49 187.96 0)
       (effects
@@
         (font
           (size 1.27 1.27)) hide))
-    (property "LCSC" "C1525"
+    (property "LCSC" "C14663"
       (at 237.49 187.96 0)
       (effects
@@
         (font
           (size 1.27 1.27))))
-    (property "Footprint" "Capacitor_SMD:C_0402_1005Metric"
+    (property "Footprint" "Capacitor_SMD:C_0603_1608Metric"
       (at 262.89 187.96 0)
       (effects
@@
         (font
           (size 1.27 1.27)) hide))
-    (property "LCSC" "C1525"
+    (property "LCSC" "C14663"
       (at 262.89 187.96 0)
       (effects
