File: hardware/lcd_board_panel.kicad_sch (KiCad schematic)
At the start: 51 parts, among them J3 AT070TN92 FPC (0.5mm 50P, top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, Q1 AO3401A, Q2 2N7002, U7 TPS61040, U8 LM321, U9 TPS61165

Commit message: Use 0603 passives and remove the alternative touch connector J6
- All 0402 resistors/capacitors are now 0603 (LCSC numbers updated to the
  matching 0603 basic parts); bulk/high-voltage caps stay 0805/1206
- J6 (JST-SH touch header) removed
- LT8619C decoupling pre-routes, crystal and REXT placement adapted to the
  larger footprints; RGB bus escape area under the chip kept free
- Re-routed (Freerouting 2.0.1), DRC: 0 errors, 0 unconnected
- Schematic, BOM/CPL, gerbers, images and README regenerated

Co-Authored-By: Claude Opus 5.5 <noreply@anthropic.com>
Claude-Session: https://claude.ai/code/session_01X8BrieHZtCS6HfoR48ML9y
Parts:
- C27, C40: footprint Capacitor_SMD:C_0402_1005Metric -> Capacitor_SMD:C_0603_1608Metric; LCSC C52923 -> C15849
- C28, C39, C41: footprint Capacitor_SMD:C_0402_1005Metric -> Capacitor_SMD:C_0603_1608Metric; LCSC C1525 -> C14663
- C30, C44: footprint Capacitor_SMD:C_0402_1005Metric -> Capacitor_SMD:C_0603_1608Metric
- C33, C36: LCSC (none) -> C14663
- C37, C38: LCSC (none) -> C15849
- R15, R16, R17, R18, R19, R20, R21: footprint Resistor_SMD:R_0402_1005Metric -> Resistor_SMD:R_0603_1608Metric; LCSC C25744 -> C25804
- R22, R23, R25, R32: footprint Resistor_SMD:R_0402_1005Metric -> Resistor_SMD:R_0603_1608Metric; LCSC C25741 -> C25803
- R24, R26, R27, R28, R29, R30: footprint Resistor_SMD:R_0402_1005Metric -> Resistor_SMD:R_0603_1608Metric
Changed lines of the file:
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@@
         (font
           (size 1.27 1.27))))
-    (property "Footprint" "Resistor_SMD:R_0402_1005Metric"
+    (property "Footprint" "Resistor_SMD:R_0603_1608Metric"
       (at 297.18 39.37 0)
       (effects
@@
         (font
           (size 1.27 1.27)) hide))
-    (property "LCSC" "C25744"
+    (property "LCSC" "C25804"
       (at 297.18 39.37 0)
       (effects
@@
         (font
           (size 1.27 1.27))))
-    (property "Footprint" "Resistor_SMD:R_0402_1005Metric"
+    (property "Footprint" "Resistor_SMD:R_0603_1608Metric"
       (at 328.93 39.37 0)
       (effects
@@
         (font
           (size 1.27 1.27)) hide))
-    (property "LCSC" "C25744"
+    (property "LCSC" "C25804"
       (at 328.93 39.37 0)
       (effects
@@
         (font
           (size 1.27 1.27))))
-    (property "Footprint" "Resistor_SMD:R_0402_1005Metric"
+    (property "Footprint" "Resistor_SMD:R_0603_1608Metric"
       (at 359.41 39.37 0)
       (effects
@@
         (font
           (size 1.27 1.27)) hide))
-    (property "LCSC" "C25744"
+    (property "LCSC" "C25804"
       (at 359.41 39.37 0)
       (effects
@@
         (font
           (size 1.27 1.27))))
-    (property "Footprint" "Resistor_SMD:R_0402_1005Metric"
+    (property "Footprint" "Resistor_SMD:R_0603_1608Metric"
       (at 30.48 181.61 0)
       (effects
@@
         (font
           (size 1.27 1.27)) hide))
-    (property "LCSC" "C25744"
+    (property "LCSC" "C25804"
       (at 30.48 181.61 0)
       (effects
@@
         (font
           (size 1.27 1.27))))
-    (property "Footprint" "Resistor_SMD:R_0402_1005Metric"
+    (property "Footprint" "Resistor_SMD:R_0603_1608Metric"
       (at 63.5 181.61 0)
       (effects
@@
         (font
           (size 1.27 1.27)) hide))
-    (property "LCSC" "C25744"
+    (property "LCSC" "C25804"
       (at 63.5 181.61 0)
       (effects
@@
         (font
           (size 1.27 1.27))))
-    (property "Footprint" "Resistor_SMD:R_0402_1005Metric"
+    (property "Footprint" "Resistor_SMD:R_0603_1608Metric"
       (at 92.71 181.61 0)
       (effects
@@
         (font
           (size 1.27 1.27)) hide))
-    (property "LCSC" "C25744"
+    (property "LCSC" "C25804"
       (at 92.71 181.61 0)
       (effects
@@
         (font
           (size 1.27 1.27))))
-    (property "Footprint" "Resistor_SMD:R_0402_1005Metric"
+    (property "Footprint" "Resistor_SMD:R_0603_1608Metric"
       (at 124.46 181.61 0)
       (effects
@@
         (font
           (size 1.27 1.27)) hide))
-    (property "LCSC" "C25744"
+    (property "LCSC" "C25804"
       (at 124.46 181.61 0)
       (effects
@@
         (font
           (size 1.27 1.27))))
-    (property "Footprint" "Capacitor_SMD:C_0402_1005Metric"
+    (property "Footprint" "Capacitor_SMD:C_0603_1608Metric"
       (at 152.4 181.61 0)
       (effects
@@
         (font
           (size 1.27 1.27)) hide))
-    (property "LCSC" "C52923"
+    (property "LCSC" "C15849"
       (at 152.4 181.61 0)
       (effects
@@
         (font
           (size 1.27 1.27))))
-    (property "Footprint" "Capacitor_SMD:C_0402_1005Metric"
+    (property "Footprint" "Capacitor_SMD:C_0603_1608Metric"
       (at 179.07 181.61 0)
       (effects
@@
         (font
           (size 1.27 1.27)) hide))
-    (property "LCSC" "C1525"
+    (property "LCSC" "C14663"
       (at 179.07 181.61 0)
       (effects
@@
         (font
           (size 1.27 1.27))))
-    (property "Footprint" "Resistor_SMD:R_0402_1005Metric"
+    (property "Footprint" "Resistor_SMD:R_0603_1608Metric"
       (at 207.01 181.61 0)
       (effects
@@
         (font
           (size 1.27 1.27)) hide))
-    (property "LCSC" "C25741"
+    (property "LCSC" "C25803"
       (at 207.01 181.61 0)
       (effects
@@
         (font
           (size 1.27 1.27))))
-    (property "Footprint" "Resistor_SMD:R_0402_1005Metric"
+    (property "Footprint" "Resistor_SMD:R_0603_1608Metric"
       (at 237.49 181.61 0)
       (effects
@@
         (font
           (size 1.27 1.27)) hide))
-    (property "LCSC" "C25741"
+    (property "LCSC" "C25803"
       (at 237.49 181.61 0)
       (effects
@@
         (font
           (size 1.27 1.27))))
-    (property "Footprint" "Resistor_SMD:R_0402_1005Metric"
+    (property "Footprint" "Resistor_SMD:R_0603_1608Metric"
       (at 337.82 181.61 0)
       (effects
@@
         (font
           (size 1.27 1.27))))
-    (property "Footprint" "Resistor_SMD:R_0402_1005Metric"
+    (property "Footprint" "Resistor_SMD:R_0603_1608Metric"
       (at 27.94 200.66 0)
       (effects
@@
         (font
           (size 1.27 1.27)) hide))
-    (property "LCSC" "C25741"
+    (property "LCSC" "C25803"
       (at 27.94 200.66 0)
       (effects
@@
         (font
           (size 1.27 1.27))))
-    (property "Footprint" "Capacitor_SMD:C_0402_1005Metric"
+    (property "Footprint" "Capacitor_SMD:C_0603_1608Metric"
       (at 59.69 200.66 0)
       (effects
@@
         (font
           (size 1.27 1.27)) hide))
-    (property "LCSC" ""
+    (property "LCSC" "C14663"
       (at 143.51 200.66 0)
       (effects
@@
         (font
           (size 1.27 1.27))))
-    (property "Footprint" "Resistor_SMD:R_0402_1005Metric"
+    (property "Footprint" "Resistor_SMD:R_0603_1608Metric"
       (at 208.28 200.66 0)
       (effects
@@
         (font
           (size 1.27 1.27)) hide))
-    (property "LCSC" ""
+    (property "LCSC" "C14663"
       (at 264.16 200.66 0)
       (effects
@@
         (font
           (size 1.27 1.27)) hide))
-    (property "LCSC" ""
+    (property "LCSC" "C15849"
       (at 295.91 200.66 0)
       (effects
@@
         (font
           (size 1.27 1.27))))
-    (property "Footprint" "Resistor_SMD:R_0402_1005Metric"
+    (property "Footprint" "Resistor_SMD:R_0603_1608Metric"
       (at 327.66 200.66 0)
       (effects
@@
         (font
           (size 1.27 1.27)) hide))
-    (property "LCSC" ""
+    (property "LCSC" "C15849"
       (at 355.6 200.66 0)
       (effects
@@
         (font
           (size 1.27 1.27))))
-    (property "Footprint" "Resistor_SMD:R_0402_1005Metric"
+    (property "Footprint" "Resistor_SMD:R_0603_1608Metric"
       (at 29.21 220.98 0)
       (effects
@@
         (font
           (size 1.27 1.27))))
-    (property "Footprint" "Resistor_SMD:R_0402_1005Metric"
+    (property "Footprint" "Resistor_SMD:R_0603_1608Metric"
       (at 100.33 220.98 0)
       (effects
@@
         (font
           (size 1.27 1.27))))
-    (property "Footprint" "Capacitor_SMD:C_0402_1005Metric"
+    (property "Footprint" "Capacitor_SMD:C_0603_1608Metric"
       (at 134.62 220.98 0)
       (effects
@@
         (font
           (size 1.27 1.27)) hide))
-    (property "LCSC" "C1525"
+    (property "LCSC" "C14663"
       (at 134.62 220.98 0)
       (effects
@@
         (font
           (size 1.27 1.27))))
-    (property "Footprint" "Resistor_SMD:R_0402_1005Metric"
+    (property "Footprint" "Resistor_SMD:R_0603_1608Metric"
       (at 168.91 220.98 0)
       (effects
@@
         (font
           (size 1.27 1.27))))
-    (property "Footprint" "Capacitor_SMD:C_0402_1005Metric"
+    (property "Footprint" "Capacitor_SMD:C_0603_1608Metric"
       (at 199.39 220.98 0)
       (effects
@@
         (font
           (size 1.27 1.27)) hide))
-    (property "LCSC" "C52923"
+    (property "LCSC" "C15849"
       (at 199.39 220.98 0)
       (effects
@@
         (font
           (size 1.27 1.27))))
-    (property "Footprint" "Capacitor_SMD:C_0402_1005Metric"
+    (property "Footprint" "Capacitor_SMD:C_0603_1608Metric"
       (at 224.79 220.98 0)
       (effects
@@
         (font
           (size 1.27 1.27)) hide))
-    (property "LCSC" "C1525"
+    (property "LCSC" "C14663"
       (at 224.79 220.98 0)
       (effects
@@
         (font
           (size 1.27 1.27))))
-    (property "Footprint" "Capacitor_SMD:C_0402_1005Metric"
+    (property "Footprint" "Capacitor_SMD:C_0603_1608Metric"
       (at 335.28 220.98 0)
       (effects
@@
         (font
           (size 1.27 1.27))))
-    (property "Footprint" "Resistor_SMD:R_0402_1005Metric"
+    (property "Footprint" "Resistor_SMD:R_0603_1608Metric"
       (at 57.15 240.03 0)
       (effects
@@
         (font
           (size 1.27 1.27)) hide))
-    (property "LCSC" "C25741"
+    (property "LCSC" "C25803"
       (at 57.15 240.03 0)
       (effects
