File: hardware/lcd_board_power.kicad_sch (KiCad schematic)
At the start: 25 parts, among them J2 USB-C (power + touch USB), U2 AMS1117-3.3, U3 AMS1117-1.8, U4 USBLC6-2SC6

Commit message: Use 0603 passives and remove the alternative touch connector J6
- All 0402 resistors/capacitors are now 0603 (LCSC numbers updated to the
  matching 0603 basic parts); bulk/high-voltage caps stay 0805/1206
- J6 (JST-SH touch header) removed
- LT8619C decoupling pre-routes, crystal and REXT placement adapted to the
  larger footprints; RGB bus escape area under the chip kept free
- Re-routed (Freerouting 2.0.1), DRC: 0 errors, 0 unconnected
- Schematic, BOM/CPL, gerbers, images and README regenerated

Co-Authored-By: Claude Opus 5.5 <noreply@anthropic.com>
Claude-Session: https://claude.ai/code/session_01X8BrieHZtCS6HfoR48ML9y
Parts:
- C2, C4: footprint Capacitor_SMD:C_0402_1005Metric -> Capacitor_SMD:C_0603_1608Metric; LCSC C1525 -> C14663
- R1, R2: footprint Resistor_SMD:R_0402_1005Metric -> Resistor_SMD:R_0603_1608Metric; LCSC C25905 -> C23186
Changed lines of the file:
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@@
         (font
           (size 1.27 1.27))))
-    (property "Footprint" "Resistor_SMD:R_0402_1005Metric"
+    (property "Footprint" "Resistor_SMD:R_0603_1608Metric"
       (at 123.19 39.37 0)
       (effects
@@
         (font
           (size 1.27 1.27)) hide))
-    (property "LCSC" "C25905"
+    (property "LCSC" "C23186"
       (at 123.19 39.37 0)
       (effects
@@
         (font
           (size 1.27 1.27))))
-    (property "Footprint" "Resistor_SMD:R_0402_1005Metric"
+    (property "Footprint" "Resistor_SMD:R_0603_1608Metric"
       (at 154.94 39.37 0)
       (effects
@@
         (font
           (size 1.27 1.27)) hide))
-    (property "LCSC" "C25905"
+    (property "LCSC" "C23186"
       (at 154.94 39.37 0)
       (effects
@@
         (font
           (size 1.27 1.27))))
-    (property "Footprint" "Capacitor_SMD:C_0402_1005Metric"
+    (property "Footprint" "Capacitor_SMD:C_0603_1608Metric"
       (at 207.01 39.37 0)
       (effects
@@
         (font
           (size 1.27 1.27)) hide))
-    (property "LCSC" "C1525"
+    (property "LCSC" "C14663"
       (at 207.01 39.37 0)
       (effects
@@
         (font
           (size 1.27 1.27))))
-    (property "Footprint" "Capacitor_SMD:C_0402_1005Metric"
+    (property "Footprint" "Capacitor_SMD:C_0603_1608Metric"
       (at 299.72 39.37 0)
       (effects
@@
         (font
           (size 1.27 1.27)) hide))
-    (property "LCSC" "C1525"
+    (property "LCSC" "C14663"
       (at 299.72 39.37 0)
       (effects
