File: hardware/lcd_board.kicad_pcb (KiCad board)
At the start: 2 copper layers, 80 x 50 mm, 126 parts, among them J1 HDMI-A receptacle, J2 USB-C (power + touch USB), J3 AT070TN92 FPC (0.5mm 50P, top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, J4 Touch FPC 6P 0.5mm, J5 SWD/UART, Q1 AO3401A, Q2 2N7002, SW1 BOOT (DFU), U1 LT8619C, U10 STM32F072CBT6, U2 AMS1117-3.3, U3 AMS1117-1.8, U4 USBLC6-2SC6, U7 TPS61040, U8 LM321, U9 TPS61165, Y1 25MHz 12pF

Commit message: Add "novin3dp.ir HDMI7" to the top silkscreen
Co-Authored-By: Claude Opus 5.5 <noreply@anthropic.com>
Claude-Session: https://claude.ai/code/session_01X8BrieHZtCS6HfoR48ML9y
Other:
- board text added: "HDMI7"
- board text added: "novin3dp.ir"
